Commit message: fix(CAD): Se ajusta los parametros de exportacion del modelo CAD a URDF

File: CAD_3D/EXPORT/little_robot_2023/urdf/little_robot_2023.urdf (robot description, URDF)
Before this commit: robot little_robot_2023, 4 links, 3 joints
Links:
- link base_link: mass 0.0777899760094901 -> 0.07779
- link link_1: mass 0.0329723164655008 -> 0.032972
- link link_2: mass 0.0311292468826037 -> 0.031129
- link link_3: mass 0.0159246060145435 -> 0.015925
Joints:
- joint joint_2: limit lower=0 upper=0 effort=0 velocity=0 -> lower=-1.572 upper=-1.572 effort=0 velocity=0
- joint joint_3: limit lower=0 upper=0 effort=0 velocity=0 -> lower=-1.572 upper=-1.572 effort=0 velocity=0

Commit message: fix(CAD): 2do ajuste a la exportacion SW to URDF

File: CAD_3D/EXPORT/little_robot_2023/urdf/little_robot_2023.urdf (robot description, URDF)
Before this commit: robot little_robot_2023, 4 links, 3 joints
Joints:
- joint joint_1: axis 0 0 -1 -> 0 0 1; origin xyz=0 0 0 rpy=0 0 0 -> xyz=0 0 0.042 rpy=3.1416 0 3.1416
- joint joint_2: axis -1 0 0 -> 0 -1 0; origin xyz=0 0 0 rpy=0 0 0 -> xyz=0 0 -0.0845 rpy=0 0 1.5708
- joint joint_3: axis -1 0 0 -> 0 0 1; origin xyz=0 0 0 rpy=0 0 0 -> xyz=0.1135 0 0 rpy=1.5708 -1.5708 0

Commit message: se ajusta el  ensamble del modelo por links para convertirlo apropiadamente a  URDF

File: CAD_3D/EXPORT/little_robot_2023/urdf/little_robot_2023.urdf (robot description, URDF)
Before this commit: robot little_robot_2023, 4 links, 3 joints
Joints:
- joint joint_1: axis 0 0 1 -> 0 1 0; limit lower=-1.572 upper=1.572 effort=0 velocity=0 -> lower=-1.571 upper=1.571 effort=0 velocity=0; origin xyz=0 0 0.042 rpy=3.1416 0 3.1416 -> xyz=0 0 0.042 rpy=1.5708 0 1.5708
- joint joint_2: axis 0 -1 0 -> 0 0 1; limit lower=-1.572 upper=-1.572 effort=0 velocity=0 -> lower=-1.571 upper=1.571 effort=0 velocity=0; origin xyz=0 0 -0.0845 rpy=0 0 1.5708 -> xyz=0 0.0845 0 rpy=0 0 0
- joint joint_3: limit lower=-1.572 upper=-1.572 effort=0 velocity=0 -> lower=-1.571 upper=1.571 effort=0 velocity=0; origin xyz=0.1135 0 0 rpy=1.5708 -1.5708 0 -> xyz=0.1135 0 0 rpy=0 0 0
